File: hardware/lcd_duffle_smd_mk_2.brd (EAGLE design)
At the start: 80 x 36 mm, 14 parts, among them IC1 ATTINY84, IC2 WS2811, J1 AVR_SPI_PRG_6TESTPOINTS, Q1 MMBT2222A

Commit message: updating libs
Parts:
- removed C4, C5: 0.1uF, A_butts:C0603
- added D1: DIODE-ZENERSOD123, A_butts:SOD123
- added Q2: MOSFET-NCHANNELIRLML2502, A_butts:SOT23
- Q1: value MMBT2222A -> MOSFET-NCHANNELIRLML2502; device SparkFun-DiscreteSemi:SOT23-3 -> A_butts:SOT23
- moved C2 22.0 mm to (9.69, 27.0), turned to 0 degrees
- moved C1 21.9 mm to (35.0, 17.0)
- moved J1 17.3 mm to (43.1, 14.5), turned to 270 degrees
- moved Q1 11.2 mm to (45.0, 23.9), turned to 270 degrees
- moved C3 6.03 mm to (59.4, 23.1)
- moved R4 3.50 mm to (57.2, 23.1), turned to 270 degrees
- moved R1 2.33 mm to (38.9, 17.0), turned to 0 degrees
- moved IC2 2.03 mm to (51.7, 22.0), turned to 270 degrees
- moved I2C 1.70 mm to (73.7, 18.0)
- moved CONTRAST 1.42 mm to (13.1, 18.0)
- moved IC1 0.94 mm to (38.0, 22.1)
Connections:
- removed net EXT_RST: C1.1, J1.5
- removed net RST: C1.2, IC1.4, R1.1
- new net N$1: D1.A, I2C.1, Q2.2
- new net RESET: IC1.4, J1.5, R1.1
- net 5V: now also C1.2, D1.C, Q2.1; no longer C3.2, C4.2, C5.2
- net GND: now also C1.1, Q2.3; no longer C4.1, C5.1, I2C.1
- net N$2: now also C3.2
Other:
- outline, holes or cut-outs redrawn
