File: hardware/lcd_duffle_smd_mk_2.sch (EAGLE design)
At the start: 14 parts, among them IC1 ATTINY84, IC2 WS2811, J1 AVR_SPI_PRG_6TESTPOINTS, Q1 MMBT2222A

Commit message: updating libs
Parts:
- removed C4, C5: 0.1uF, A_butts:CAPACITOR-CERAMICC0603
- added D1: DIODE-ZENERSOD123, A_butts:DIODE-ZENERSOD123
- added Q2: MOSFET-NCHANNELIRLML2502, A_butts:MOSFET-NCHANNELIRLML2502
- Q1: value MMBT2222A -> MOSFET-NCHANNELIRLML2502; device SparkFun-DiscreteSemi:TRANSISTOR_NPNMMBT2222A -> A_butts:MOSFET-NCHANNELIRLML2502
Connections:
- removed net EXT_RST: C1.1, J1.5
- removed net RST: C1.2, IC1.(PCINT11/~RESET/DW)PB3, R1.1
- new net N$1: D1.A, I2C.1, Q2.S
- new net RESET: IC1.(PCINT11/~RESET/DW)PB3, J1.5, R1.1
- net 5V: now also C1.2, D1.C, Q2.G; no longer C3.2, C4.2, C5.2
- net GND: now also C1.1, Q1.S, Q2.D; no longer C4.1, C5.1, I2C.1, Q1.E
- net LED_CNTL: now also Q1.G; no longer Q1.B
- net N$2: now also C3.2
- net R: now also Q1.D; no longer Q1.C
Other:
- moved on the sheet: C1, C2, C3, I2C
