File: hardware/lcd_duffle_smd_mk_3.sch (EAGLE design)
At the start: 15 parts, among them IC1 ATTINY84, IC2 WS2811

Commit message: wooo
Parts:
- removed AVRISP: AVR_SPI_PRG_6SMD-M-RA, A_butts:AVR_SPI_PRG_6SMD-M-RA
- removed D2: MBRA140, A_butts:DIODE-SCHOTTKYMBRA140
- removed I2C: I2C, A_butts:M04SMD
- added JP1: M06SMD, A_butts:M06SMD
- added MONOCHROME?: JUMPER-PAD-2-NOYES_SILK, A_butts:JUMPER-PAD-2-NOYES_SILK
Connections:
- removed net LED_CNTL: AVRISP.MISO, IC1.(PCINT5/OC1B/MISO/DO/ADC5)PA5, IC2.DIN
- removed net N$3: AVRISP.VCC, D2.C
- new net LIGHT: IC1.(PCINT7/ICP/OC0B/ADC7)PA7, IC2.DIN, MONOCHROME?.2
- new net MISO: IC1.(PCINT5/OC1B/MISO/DO/ADC5)PA5, JP1.2
- net 5V: no longer D2.A
- net E: now also IC1.(PCINT10/INT0/OC0A/CKOUT)PB2; no longer IC1.(PCINT7/ICP/OC0B/ADC7)PA7
- net GND: now also JP1.6; no longer AVRISP.GND, I2C.1, U$1.DB0, U$1.DB1, U$1.DB2, U$1.DB3
- net N$1: now also JP1.5; no longer I2C.4
- net R: now also MONOCHROME?.1
- net RESET: now also JP1.1; no longer AVRISP.RESET
- net RS: now also IC1.(PCINT8/XTAL1/CLKI)PB0; no longer IC1.(PCINT9/XTAL2)PB1
- net RW: now also IC1.(PCINT9/XTAL2)PB1; no longer IC1.(PCINT10/INT0/OC0A/CKOUT)PB2
- net SCL: now also JP1.4; no longer AVRISP.SCK, I2C.2
- net SDA: now also JP1.3; no longer AVRISP.MOSI, I2C.3
Other:
- note removed: "Use the WS2811 for RGB-backlight LCDs (18 pin) Use NPN transistor (2N3904, 2N2222A) for single-color backlight LCDs (16 pin)"
- moved on the sheet: D1

Commit message: ready for the fab
Parts:
- added R5: (no value), A_butts:RESISTORR0805
- CONTRAST: device A_butts:POTENTIOMETERTHUMBWHEEL-16MM -> A_butts:POTENTIOMETER3314Z
Connections:
- net CONTRAST: now also R5.1
- net GND: now also R5.2
Other:
- note added: "Set contrast permanently by populating R5 (ballpark 1-2k?)"
- moved on the sheet: CONTRAST
