File: hardware/lcd_buckler_mk_2.sch (EAGLE design)
At the start: 16 parts, among them IC1 ATTINY84

Commit message: version 2 ready for fab. added lcd connections and trimpots to both sides in case i need to reverse/flip something. disconnect for i2c pull-ups as i'm wondering if those are causing problems.
Parts:
- removed CONTRAST1: 10k, A_butts:POTENTIOMETERTHUMBWHEEL-16MM
- removed LCD: LCD-16x2, A_butts:LCD-16X2HOLESONLY
- added CONTRAST_L, CONTRAST_R: 10k, A_butts:POTENTIOMETERTHUMBWHEEL-16MM
- added LCD_BOTTOM, LCD_TOP: LCD-16x2, A_butts:LCD-16X2HOLESONLY
- renumbered JP1 to PULLUP_I2C?
Connections:
- net 5V: now also CONTRAST_L.E, CONTRAST_R.E, LCD_BOTTOM.A, LCD_BOTTOM.VDD, LCD_TOP.A, LCD_TOP.VDD; no longer CONTRAST1.E, LCD.A, LCD.VDD
- net BACKLIGHT: now also LCD_BOTTOM.K, LCD_TOP.K; no longer LCD.K
- net CON: now also CONTRAST_L.S, CONTRAST_R.S, LCD_BOTTOM.VO, LCD_TOP.VO; no longer CONTRAST1.S, LCD.VO
- net DB4: now also LCD_BOTTOM.DB4, LCD_TOP.DB4; no longer LCD.DB4
- net DB5: now also LCD_BOTTOM.DB5, LCD_TOP.DB5; no longer LCD.DB5
- net DB6: now also LCD_BOTTOM.DB6, LCD_TOP.DB6; no longer LCD.DB6
- net DB7: now also LCD_BOTTOM.DB7, LCD_TOP.DB7; no longer LCD.DB7
- net E: now also LCD_BOTTOM.E, LCD_TOP.E; no longer LCD.E
- net GND: now also CONTRAST_L.A, CONTRAST_R.A, LCD_BOTTOM.VSS, LCD_TOP.VSS; no longer CONTRAST1.A, LCD.VSS
- net RS: now also LCD_BOTTOM.RS, LCD_TOP.RS; no longer LCD.RS
- net RW: now also LCD_BOTTOM.R/W, LCD_TOP.R/W; no longer LCD.R/W
