File: hardware/lcd_buckler_mk_1.brd (EAGLE design)
At the start: 52 x 43 mm, 16 parts, among them IC1 ATTINY84

Commit message: updates for the update throne
Connections:
- net MOSISDA renamed MOSI/SDA
Changed lines of the file:
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@@
 <setting verticaltext="up"/>
 </settings>
-<grid distance="0.1" unitdist="mm" unit="mm" style="lines" multiple="5" display="yes" altdistance="1" altunitdist="mil" altunit="mil"/>
+<grid distance="0.5" unitdist="mm" unit="mm" style="lines" multiple="2" display="yes" altdistance="1" altunitdist="mil" altunit="mil"/>
 <layers>
 <layer number="1" name="Top" color="4" fill="1" visible="yes" active="yes"/>
@@
 <wire x1="16.6" y1="19.71" x2="16.6" y2="3.49" width="0.25" layer="16"/>
 </signal>
-<signal name="MOSISDA">
+<signal name="MOSI/SDA">
 <contactref element="SHIELD" pad="A4"/>
 <contactref element="R2" pad="P$1"/>
