File: hardware/lcd_buckler_mk_1.sch (EAGLE design)
At the start: 11 parts, among them IC1 ATTINY84

Commit message: updates for the update throne
Connections:
- net MOSISDA renamed MOSI/SDA
Changed lines of the file:
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@@
 </segment>
 </net>
-<net name="MOSISDA" class="0">
+<net name="MOSI/SDA" class="0">
 <segment>
 <pinref part="SHIELD" gate="G$1" pin="A4"/>
